File: PCB dos canales/PCB dos canales.kicad_sch (KiCad schematic)
At the start: 74 parts

Commit message: Gustavo agrega cambios en la pcb dos canales
Parts:
- removed RV? (x2): 100K, Potentiometer_THT:Potentiometer_Bourns_3296W_Vertical, symbol Device:R_Potentiometer_Trim
- added unit 1 of U6
- added unit 5 of U6
- C1: renamed from C?; value 47uF -> (none); footprint Capacitor_THT:CP_Radial_D5.0mm_P2.50mm -> (none)
- C10, C11, C14, C15: renamed from C?; value 1uF -> (none); footprint Capacitor_THT:C_Disc_D5.0mm_W2.5mm_P5.00mm -> (none)
- C13, C4: renamed from C?; value 220nF -> (none); footprint Capacitor_THT:C_Disc_D5.0mm_W2.5mm_P5.00mm -> (none)
- C9: renamed from C?; value 1nF -> (none); footprint Capacitor_SMD:C_1206_3216Metric -> (none)
- J1, J2: renamed from J?; value Conn_01x02 -> (none); footprint TerminalBlock_Phoenix:TerminalBlock_Phoenix_MKDS-1,5-2_1x02_P5.00mm_Horizontal -> (none)
- J3: renamed from J?; value Conn_01x03 -> (none); footprint TerminalBlock_Phoenix:TerminalBlock_Phoenix_MKDS-1,5-3-5.08_1x03_P5.08mm_Horizontal -> (none)
- R11, R15, R25, R31: renamed from R?; value 1M -> (none); footprint Resistor_THT:R_Axial_DIN0207_L6.3mm_D2.5mm_P10.16mm_Horizontal -> (none)
- R13, R3, R6, R9: renamed from R?; value 39K -> (none); footprint Resistor_THT:R_Axial_DIN0207_L6.3mm_D2.5mm_P10.16mm_Horizontal -> (none)
- R2: renamed from R?; value 2.2M -> (none); footprint Resistor_THT:R_Axial_DIN0207_L6.3mm_D2.5mm_P10.16mm_Horizontal -> (none)
- R22, R29: renamed from R?; value 560K -> (none); footprint Resistor_THT:R_Axial_DIN0207_L6.3mm_D2.5mm_P10.16mm_Horizontal -> (none)
- R7: renamed from R?; value 4.7K -> (none); footprint Resistor_SMD:R_1206_3216Metric -> (none)
- U1, U2: renamed from U?; value AD620 -> (none); footprint Package_DIP:DIP-8_W7.62mm -> (none)
- U3, U5: renamed from U?; value LM324 -> (none); footprint Package_SO:SO-14_3.9x8.65mm_P1.27mm -> (none)
- U4, U6: renamed from U?; value LM324 -> (none); footprint Package_DIP:DIP-14_W7.62mm_Socket -> (none)
- gave numbers to parts that had none: 29
Connections:
- net +V: now also U6.4 (V+)
- net -V: now also U6.11 (V-)
- net at R30.2, U3.9 (-): now also R32.2
- net at R23.2, U5.9 (-): now also R28.2
- no-connect marks 8 -> 9
Other:
- note added: "A: Filtro de RFI (Horizontal)"
- note added: "A: Filtro de RFI (Vertical)"
- note added: "B: Adquisicion de señal (Horizontal)"
- note added: "B: Adquisicion de señal (Vertical)"
- note added: "CIRCUITO DE RECHADO DE MODO COMUN (Horizontal)"
- note added: "CIRCUITO DE RECHADO DE MODO COMUN (Vertical)"
- note added: "D: Etapa de amplificacion principal (Horizontal)"
- note added: "D: Etapa de amplificacion principal (Vertical)"
- note added: "E: Filtro pasa banda de segundo orden (Horizontal)"
- note added: "E: Filtro pasa banda de segundo orden (Vertical)"
- note added: "F: Amplificador variable (Horizontal)"
- note added: "F: Amplificador variable (Vertical)"
- note added: "Operacionales sin conexion"
- note removed: "A: Filtro de RFI"
- note removed: "B: Adquisicion de señal"
- note removed: "CIRCUITO DE RECHADO DE MODO COMUN"
- note removed: "D: Etapa de amplificacion principal"
- note removed: "E: Filtro pasa banda de segundo orden"
- note removed: "F: Amplificador variable"
- moved on the sheet: C10, C11, C2, C3, C4, C5, C6, R10, R11, R12, R17, R18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
